Commit message: temp

File: source/DoorOpening/assets/door/PartNet/8893/mobility.urdf (robot description, URDF)
Before this commit: robot partnet_24ef5084512256551bffd4bc88cc8d80, 4 links, 3 joints
Joints:
- joint joint_1: origin xyz=0.6663215063128132 -0.8974214251025738 -0.022139757071257815 -> xyz=0.6663215063128132 -0.8974214251025738 -0.042139757071257815
