Commit message: cubic spline

File: source/DoorOpening/assets/door/PartNetv2/99650069960003/mobility.urdf (robot description, URDF)
Before this commit: robot right-pull-door, 4 links, 3 joints
Links:
- link link_0: geometry collision mesh filename=texture_dae/frame.obj scale=0.8200447754284704 0.8200447754284704 0.8200447754284704; visual mesh filename=texture_dae/frame.obj scale=0.8200447754284704 0.8200447754284704 0.8200447754284704

Commit message: introduce door pos err reward

File: source/DoorOpening/assets/door/PartNetv2/99650069960003/mobility.urdf (robot description, URDF)
Before this commit: robot right-pull-door, 4 links, 3 joints
Joints:
- joint joint_2: origin xyz=0.6698489351830481 -0.9444402274483152 0.04279544730454047 -> xyz=0.6698489351830481 -0.9444402274483152 0.0
