Commit message: first attempt

File: source/DoorOpening/assets/door/PartNetv2/99650069962004/mobility.urdf (robot description, URDF)
Before this commit: robot right-pull-door, 4 links, 3 joints
Joints:
- joint joint_1: limit lower=0 upper=1.5079644737231006 -> lower=-1.5079644737231006 upper=0

Commit message: some updates

File: source/DoorOpening/assets/door/PartNetv2/99650069962004/mobility.urdf (robot description, URDF)
Before this commit: robot right-pull-door, 4 links, 3 joints
Joints:
- joint joint_1: limit lower=-1.5079644737231006 upper=0 -> lower=0 upper=1.5079644737231006
