Commit message: checkpoint

File: source/DoorOpening/assets/glorbot/glorbot.urdf (robot description, URDF)
Before this commit: robot tidybot2, 58 links, 57 joints
Links:
- link back_right_steer_link: mass 0 -> 0.23041

Commit message: dr update

File: source/DoorOpening/assets/glorbot/glorbot.urdf (robot description, URDF)
Before this commit: robot tidybot2, 58 links, 57 joints
Links:
- link back_right_steer_link: mass 0.23041 -> 0
