Commit message: RL improvement

File: source/DoorOpening/assets/glorbot/glorbot.urdf (robot description, URDF)
Before this commit: robot tidybot2, 58 links, 57 joints
Links:
- link tidybot2_base_link: geometry collision mesh filename=package://glorbot/meshes/tidybot2/tidybot2_base_link.STL; visual mesh filename=package://glorbot/meshes/tidybot2/tidybot2_base_link.STL

Commit message: update collisiong

File: source/DoorOpening/assets/glorbot/glorbot.urdf (robot description, URDF)
Before this commit: robot tidybot2, 58 links, 57 joints
Links:
- link lidar: geometry collision box size=0.103 0.075 0.148; visual mesh filename=package://glorbot/meshes/tidybot2/lidar.STL
- link link3: geometry collision mesh filename=package://glorbot/meshes/arx_x5/link3.STL; visual mesh filename=package://glorbot/meshes/arx_x5/link3.STL
- link link4: geometry collision mesh filename=package://glorbot/meshes/arx_x5/link4.STL; visual mesh filename=package://glorbot/meshes/arx_x5/link4.STL
- link link5: geometry collision mesh filename=package://glorbot/meshes/arx_x5/link5.STL; visual mesh filename=package://glorbot/meshes/arx_x5/link5.STL
- link palm_lower: geometry collision mesh filename=package://glorbot/meshes/leap/palm_lower.stl; visual mesh filename=package://glorbot/meshes/leap/palm_lower.stl
- link panda_link5: geometry collision mesh filename=package://glorbot/meshes/franka/visual/link5.obj; visual mesh filename=package://glorbot/meshes/franka/visual/link5.obj
- link tidybot2_base_link: geometry collision mesh filename=package://glorbot/meshes/tidybot2/tidybot2_mast.STL; visual mesh filename=package://glorbot/meshes/tidybot2/tidybot2_base_link.STL

Commit message: update base vel

File: source/DoorOpening/assets/glorbot/glorbot.urdf (robot description, URDF)
Before this commit: robot tidybot2, 58 links, 57 joints
Links:
- link dip_4: geometry collision box size=0.01 0.024 0.018; collision box size=0.014 0.02 0.004
- link fingertip_4: geometry collision box size=0.008 0.024 0.018; collision box size=0.02 0.004 0.03
- link mcp_joint_4: geometry collision box size=0.034 0.026 0.022; visual mesh filename=package://glorbot/meshes/leap/pip.stl
- link palm_lower: geometry collision box size=0.004 0.036 0.034; collision box size=0.01 0.12 0.02
- link pip_4: geometry collision box size=0.014 0.004 0.02; collision box size=0.014 0.004 0.02

Commit message: fix finger tip urdf + unlatching

File: source/DoorOpening/assets/glorbot/glorbot.urdf (robot description, URDF)
Before this commit: robot tidybot2, 58 links, 57 joints
Links:
- link fingertip_4: geometry collision mesh filename=package://glorbot/meshes/leap/thumb_fingertip.stl; visual mesh filename=package://glorbot/meshes/leap/thumb_fingertip_color.obj
