Commit message: Replace the LEAP hand with Franka's 2-finger gripper throughout
The robot IS the gripper on this branch: no parallel *_gripper files, no LEAP
code path left to choose between. glorbot.urdf, glorbot_cfg.py,
slider_controller.py and hard_code_traj.py keep their names and their exported
symbols (GLORBOT_CONFIG, DEFAULT_JOINT_POS, FULL_JOINT_NAMES,
OmniJointController, ...), so consumers are updated in place rather than
forked.

Robot: the LEAP block (palm_lower, 16 finger_joint_*, realtip_*) is replaced by
the stock Panda hand -- panda_link8 at z=0.107 off link7, panda_hand yawed
-45 deg, two prismatic fingers. 18 DOFs instead of 31. palm_center is retained
as the end-effector frame name, now at the stock TCP, which the Franka Hand
manual's flange->TCP transform (pz=0.1034, -45 deg) confirms.

One commanded DOF, like the real single-actuator hand: panda_finger_joint2
mimics joint1. HONOR_URDF_MIMIC picks between the PhysX mimic constraint
(requires convert_mimic_joints_to_normal_joints=True, whose name is inverted
relative to what it does) and a software-coupled fallback. FULL_JOINT_NAMES
therefore carries one finger entry; ALL_DOF_NAMES is the full 18 when a whole
joint-state tensor is needed.

Drive parameters come from the Franka Hand Product Manual (R50010 v1.2, 5.1):
effort 70 N (30-70 N continuous band), velocity 0.05 m/s (50 mm/s per finger,
4x slower than the 0.2 everyone copies from Isaac Lab), stiffness 5e3 so a
full-close on a ~20 mm handle lands mid-band at ~50 N, damping 60 for zeta >= 1
in both coupling modes, armature 0.05 kg so 15 g fingers cannot cross their
travel inside one step.

Task layer follows: the action space's finger block goes 12 -> 1, contact
sensors move to panda_hand / the two fingers, the self-collision hand group
becomes the fingers vs the flange, the armature ADR term is rescoped and given
a mass-valued nominal, the IK end-effector link becomes panda_hand, and the
collision checker's sphere model is rebuilt for the hand. NOTE this changes the
action space, so LEAP-trained checkpoints will not load against this robot.

glorbot_wheels.urdf is deliberately left untouched, LEAP hand and all: nothing
imports it, so it is inert here and is kept as-is rather than ported or dropped.

Removed as dead: utils/finger_utils.py (LEAP tendon math) and a TEMP
abduction-clamp diagnostic in multi_dooropening_env.py that was marked "revert
before commit". FrankaLeapSampler is renamed FrankaGripperSampler.

Co-Authored-By: Claude Opus 5 <noreply@anthropic.com>

File: source/DoorOpening/assets/glorbot/glorbot.urdf (robot description, URDF)
Before this commit: robot tidybot2, 58 links, 57 joints
Links:
- removed link dip_1
- removed link dip_2
- removed link dip_3
- removed link dip_4
- removed link fingertip_1
- removed link fingertip_2
- removed link fingertip_3
- removed link fingertip_4
- removed link mcp_joint_1
- removed link mcp_joint_2
- removed link mcp_joint_3
- removed link mcp_joint_4
- removed link palm_lower
- removed link pip_1
- removed link pip_2
- removed link pip_3
- removed link pip_4
- removed link realtip_1
- removed link realtip_2
- removed link realtip_3
- removed link realtip_4
- added link left_fingertip
- added link panda_hand, mass 0.73; collision mesh filename=package://glorbot/meshes/franka/collision/hand.obj; visual mesh filename=package://glorbot/meshes/franka/visual/hand.obj
- added link panda_leftfinger, mass 0.015; collision mesh filename=package://glorbot/meshes/franka/collision/finger.obj; visual mesh filename=package://glorbot/meshes/franka/visual/finger.obj
- added link panda_link8
- added link panda_rightfinger, mass 0.015; collision mesh filename=package://glorbot/meshes/franka/collision/finger.obj; visual mesh filename=package://glorbot/meshes/franka/visual/finger.obj
- added link right_fingertip
Joints:
- removed joint finger_joint_0
- removed joint finger_joint_1
- removed joint finger_joint_10
- removed joint finger_joint_11
- removed joint finger_joint_12
- removed joint finger_joint_13
- removed joint finger_joint_14
- removed joint finger_joint_15
- removed joint finger_joint_2
- removed joint finger_joint_3
- removed joint finger_joint_4
- removed joint finger_joint_5
- removed joint finger_joint_6
- removed joint finger_joint_7
- removed joint finger_joint_8
- removed joint finger_joint_9
- removed joint tip_joint_1
- removed joint tip_joint_2
- removed joint tip_joint_3
- removed joint tip_joint_4
- added joint left_fingertip_joint: type fixed, parent panda_leftfinger, child left_fingertip, origin xyz=0 0 0.045 rpy=0 0 0
- added joint panda_finger_joint1: type prismatic, parent panda_hand, child panda_leftfinger, origin xyz=0 0 0.0584 rpy=0 0 0, axis 0 1 0, limit lower=0.0 upper=0.04 effort=70 velocity=0.05
- added joint panda_finger_joint2: type prismatic, parent panda_hand, child panda_rightfinger, origin xyz=0 0 0.0584 rpy=0 0 0, axis 0 -1 0, limit lower=0.0 upper=0.04 effort=70 velocity=0.05, mimic joint=panda_finger_joint1 multiplier=1.0 offset=0.0
- added joint panda_joint8: type fixed, parent panda_link7, child panda_link8, origin xyz=0 0 0.107 rpy=0 0 0
- added joint right_fingertip_joint: type fixed, parent panda_rightfinger, child right_fingertip, origin xyz=0 0 0.045 rpy=0 0 0
- joint palm_center_joint: child palm_lower -> palm_center; origin xyz=0.065 -0.035 0 rpy=3.14159 0 0 -> xyz=0 0 0.1034 rpy=0 0 0; parent palm_center -> panda_hand
- joint panda_hand_joint: child palm_center -> panda_hand; origin xyz=0 0 0.115 rpy=0 0 0 -> xyz=0 0 0 rpy=0 0 -0.7853981633974483; parent panda_link7 -> panda_link8

Commit message: Separate base/arm motion in left pull planner, track handle joint angle, and tune escutcheon plate/frame door-gen parameters
- offline_pull_door.py: rewrite left-door pregrasp/release/unlatch steps to
  never move base+arm simultaneously; make unlatch wrist pitch and Step 4's
  pull sweep track the actual lever joint angle (plus a small anti-slip
  margin) instead of independently tuned endpoints; unify pregrasp/pull-open
  base tilt into one constant.
- compute_waypoint.py: switch segment interpolation from a clamped cubic
  spline to PCHIP to stop overshoot on the new hold-then-move waypoint
  patterns; drop the now-dead panel_contact_mask.
- multi_motion_lib.py / multi_dooropening_env.py: remove panel_contact_mask
  plumbing; replace the per-env ADR-randomized door latch threshold with a
  fixed DOOR_LATCH_HINGE_THRESHOLD_RAD so every door requires a full press
  before the panel unlocks.
- multi_dooropening_env_cfg.py: drop the now-unused door_latch_threshold_*
  ADR range fields.
- glorbot.urdf: revert finger collision back to the dedicated collision mesh.
- generate_randomized_doors_scratch.py: widen escutcheon plate size/
  protrusion ranges, adjust handle stem-length range and
  MIN_HANDLE_PLATE_GRASP_GAP_M.
- eval_multi_distillation.py: fix reference to the removed per-env latch
  threshold tensor.

Co-Authored-By: Claude Sonnet 5 <noreply@anthropic.com>
Claude-Session: https://claude.ai/code/session_01BGzQ7GVrUvb7nQxFWSCbMH

File: source/DoorOpening/assets/glorbot/glorbot.urdf (robot description, URDF)
Before this commit: robot tidybot2, 43 links, 42 joints
Links:
- link panda_leftfinger: geometry collision mesh filename=package://glorbot/meshes/franka/collision/finger.obj; visual mesh filename=package://glorbot/meshes/franka/visual/finger.obj
- link panda_rightfinger: geometry collision mesh filename=package://glorbot/meshes/franka/collision/finger.obj; visual mesh filename=package://glorbot/meshes/franka/visual/finger.obj

Commit message: Revert fingertip collision to visual mesh, tune left pull planner offsets to match
- glorbot.urdf: panda_leftfinger/rightfinger collision back to the visual
  mesh (not the dedicated hull), matching the real L-shaped finger geometry
  discovered while testing on the new door batch.
- offline_pull_door.py: with accurate finger collision, real pad contact
  only exists in the last ~18mm near the tip, so grasp/pull now approach
  lower (grasp_palm_z_offset, pull_palm_z_offset) and slightly further from
  the panel (grasp_palm_x_offset, pull_palm_x_offset_closed) to seat the
  handle bar correctly without penetrating the panel.

Co-Authored-By: Claude Sonnet 5 <noreply@anthropic.com>
Claude-Session: https://claude.ai/code/session_01BGzQ7GVrUvb7nQxFWSCbMH

File: source/DoorOpening/assets/glorbot/glorbot.urdf (robot description, URDF)
Before this commit: robot tidybot2, 43 links, 42 joints
Links:
- link panda_leftfinger: geometry collision mesh filename=package://glorbot/meshes/franka/visual/finger.obj; visual mesh filename=package://glorbot/meshes/franka/visual/finger.obj
- link panda_rightfinger: geometry collision mesh filename=package://glorbot/meshes/franka/visual/finger.obj; visual mesh filename=package://glorbot/meshes/franka/visual/finger.obj
